File: Trigger.kicad_pcb (KiCad board)
At the start: 2 copper layers, 49.1 x 49 mm, 32 parts, among them J1 USB_B, J2 TP1, J3 Conn_01x04_IO, J4 Screw_Terminal_01x06, J5 Conn_01x05_Male, Q1 Q_NMOS_GSD, SW2 SW_Push, U1 MCP6002, U2 SAMD21E, U3 TPS769XX

Commit message: Routed!
Connections:
- J4 pad 3: /Shutter -> /Flash
- J4 pad 4: /Flash -> /Shutter
Routing:
- net GND: track 0.00 -> 212.0 mm, vias 0 -> 6
- net /3V3: track 0.00 -> 159.9 mm
- net /5V: track 0.00 -> 81.6 mm, vias 0 -> 2
- net Net-(C6-Pad1): track 0.00 -> 25.0 mm
- net /ManTrig: track 0.00 -> 23.9 mm, vias 0 -> 2
- net /RstN: track 0.00 -> 22.9 mm, vias 0 -> 2
- net Net-(R2-Pad2): track 0.00 -> 21.1 mm, vias 0 -> 2
- net /Trig: track 0.00 -> 21.0 mm
- net /Shutter: track 0.00 -> 18.7 mm
- net Net-(C6-Pad2): track 0.00 -> 18.1 mm, vias 0 -> 1
- net /Flash: track 0.00 -> 17.6 mm
- net /D1: track 0.00 -> 17.2 mm
- net /D2: track 0.00 -> 15.7 mm
- net /D3: track 0.00 -> 14.4 mm
- net /DP: track 0.00 -> 12.7 mm
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- added copper zone on B.Cu, net GND
Other:
- net class Default: trace_width 0.25 -> 0.4; via_dia 0.8 -> 0.6; via_drill 0.4 -> 0.3
- net class Pwr added: clearance 0.2, trace_width 1.5, via_dia 0.8, via_drill 0.4
- rule via_min_drill: 0.3 -> 0
- rule via_min_size: 0.4 -> 0.55
- board text added: "16"
- board text added: "17"
- board text added: "18"
- board text added: "3"
- board text added: "3v3"
- board text added: "5"
- board text added: "Clk"
- board text added: "DIO"
- board text added: "F"
- board text added: "G"
- board text added: "Gnd"
- board text added: "K"
- board text added: "PA"
- board text added: "Rst"
- board text added: "SW"
- board text added: "Sh"
- board text added: "TP"
- board text removed: "TODOs: Move refs where can be seen. Mark diode K or A Align holes Move GPIO out to other side and add more?"
