File: Trigger.sch (KiCad schematic (older format))
At the start: 32 parts, among them U1 MCP6002, U2 SAMD21E, U3 TPS769XX

Commit message: all connections made
Parts:
- added J2: TP1, symbol Connector:Conn_01x01_Male
- gave numbers to parts that had none: 24
Connections:
- net Flash: now also U2.11 (PA08)
- net ManTrig: now also U2.3 (PA02)
- net Trig: now also R2.1, R4.2, U1.7, U2.1 (PA00); no longer J4.3 (Pin_3)
- net at C6.1, R1.1, U1.1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: now also J2.1 (Pin_1)
- net Shutter: now reaches U2.12 (PA09)
- net Shutter: now also J4.3 (Pin_3)
- net D1: now reaches U2.17 (PA16)
- net D1: now also J3.2 (Pin_2)
- net at R5.1, R6.2: now also U2.20 (PA19); no longer U2.18 (PA17)
- net D3: now reaches U2.19 (PA18)
- net D3: now also J3.4 (Pin_4)
- net D2: now reaches J3.3 (Pin_3)
- net D2: now also U2.18 (PA17)
- no-connect marks 2 -> 18
Other:
- note removed: "To some GPIO"
Changed lines of the file:
@@
 	4150 2500 4150 2550
 $Comp
-L Device:LED D?
+L Device:LED D4
 U 1 1 5C3A7D51
 P 10400 1000
-F 0 "D?" V 10438 883 50  0000 R CNN
+F 0 "D4" V 10438 883 50  0000 R CNN
 F 1 "LED" V 10347 883 50  0000 R CNN
 F 2 "" H 10400 1000 50  0001 C CNN
@@
 $EndComp
 $Comp
-L Device:R R?
+L Device:R R7
 U 1 1 5C3A7E03
 P 10150 850
-F 0 "R?" V 9943 850 50  0000 C CNN
+F 0 "R7" V 9943 850 50  0000 C CNN
 F 1 "10K" V 10034 850 50  0000 C CNN
 F 2 "" V 10080 850 50  0001 C CNN
@@
 Connection ~ 9900 1150
 $Comp
-L Connector:USB_B_Micro J?
+L Connector:USB_B_Micro J1
 U 1 1 5C3A96B5
 P 1150 3600
-F 0 "J?" H 1205 4067 50  0000 C CNN
+F 0 "J1" H 1205 4067 50  0000 C CNN
 F 1 "USB_B_Micro" H 1205 3976 50  0000 C CNN
 F 2 "" H 1300 3550 50  0001 C CNN
@@
 	3750 2550 4150 2550
 $Comp
-L Switch:SW_SPST SW?
+L Switch:SW_SPST SW1
 U 1 1 5C3AFA00
 P 4500 2400
-F 0 "SW?" V 4454 2498 50  0000 L CNN
+F 0 "SW1" V 4454 2498 50  0000 L CNN
 F 1 "SW_SPST" V 4545 2498 50  0000 L CNN
 F 2 "" H 4500 2400 50  0001 C CNN
@@
 	4500 2650 4500 2600
 $Comp
-L Device:R R?
+L Device:R R3
 U 1 1 5C3B11DD
 P 5200 2400
-F 0 "R?" H 5130 2354 50  0000 R CNN
+F 0 "R3" H 5130 2354 50  0000 R CNN
 F 1 "10K" H 5130 2445 50  0000 R CNN
 F 2 "" V 5130 2400 50  0001 C CNN
@@
 Connection ~ 2400 6600
 $Comp
-L Device:C_Small C?
+L Device:C_Small C6
 U 1 1 5C3A374A
 P 2400 5550
-F 0 "C?" V 2171 5550 50  0000 C CNN
+F 0 "C6" V 2171 5550 50  0000 C CNN
 F 1 "1n" V 2262 5550 50  0000 C CNN
 F 2 "" H 2400 5550 50  0001 C CNN
@@
 $EndComp
 $Comp
-L Device:R R?
+L Device:R R1
 U 1 1 5C3A37C4
 P 2400 5200
-F 0 "R?" V 2193 5200 50  0000 C CNN
+F 0 "R1" V 2193 5200 50  0000 C CNN
 F 1 "100k" V 2284 5200 50  0000 C CNN
 F 2 "" V 2330 5200 50  0001 C CNN
@@
 Position so can\nresolder
 $Comp
-L Device:D_Photo D?
+L Device:D_Photo D1
 U 1 1 5C3A7AE6
 P 1500 6200
-F 0 "D?" V 1404 6357 50  0000 L CNN
+F 0 "D1" V 1404 6357 50  0000 L CNN
 F 1 "D_Photo" V 1495 6357 50  0000 L CNN
 F 2 "" H 1450 6200 50  0001 C CNN
@@
 	1950 5900 1950 5550
 $Comp
-L Device:R_POT RV?
+L Device:R_POT RV1
 U 1 1 5C3AA8E4
 P 3650 6000
-F 0 "RV?" H 3580 6046 50  0000 R CNN
+F 0 "RV1" H 3580 6046 50  0000 R CNN
 F 1 "20k" H 3580 5955 50  0000 R CNN
 F 2 "" H 3650 6000 50  0001 C CNN
@@
 $EndComp
 $Comp
-L Device:R R?
+L Device:R R4
 U 1 1 5C3ADF29
 P 5550 6200
-F 0 "R?" V 5343 6200 50  0000 C CNN
+F 0 "R4" V 5343 6200 50  0000 C CNN
 F 1 "220R" V 5434 6200 50  0000 C CNN
 F 2 "" V 5480 6200 50  0001 C CNN
@@
 $EndComp
 $Comp
-L Device:LED D?
+L Device:LED D2
 U 1 1 5C3AE0B1
 P 5800 6400
-F 0 "D?" V 5838 6283 50  0000 R CNN
+F 0 "D2" V 5838 6283 50  0000 R CNN
 F 1 "LED" V 5747 6283 50  0000 R CNN
 F 2 "" H 5800 6400 50  0001 C CNN
@@
 Wire Wire Line
 	4900 6200 4900 5550
-Text Notes 5050 5500 0    50   ~ 0
+Text Notes 5000 5600 0    50   ~ 0
 To Interupt
 Connection ~ 4300 6600
@@
 	3650 5800 4300 5800
 $Comp
-L Device:R R?
+L Device:R R2
 U 1 1 5C3C782D
 P 4350 5550
-F 0 "R?" V 4143 5550 50  0000 C CNN
+F 0 "R2" V 4143 5550 50  0000 C CNN
 F 1 "100k" V 4234 5550 50  0000 C CNN
 F 2 "" V 4280 5550 50  0001 C CNN
@@
 RstN
 $Comp
-L MyComponents:MountHole H?
+L MyComponents:MountHole H1
 U 1 1 5C3B6A60
 P 650 7700
-F 0 "H?" H 790 7953 60  0000 L CNN
+F 0 "H1" H 790 7953 60  0000 L CNN
 F 1 "MountHole" H 790 7847 60  0000 L CNN
 F 2 "" H 650 7700 60  0001 C CNN
@@
 $EndComp
 $Comp
-L MyComponents:MountHole H?
+L MyComponents:MountHole H2
 U 1 1 5C3B6B94
 P 1000 7700
-F 0 "H?" H 1140 7953 60  0000 L CNN
+F 0 "H2" H 1140 7953 60  0000 L CNN
 F 1 "MountHole" H 1140 7847 60  0000 L CNN
 F 2 "" H 1000 7700 60  0001 C CNN
@@
 $EndComp
 $Comp
-L MyComponents:MountHole H?
+L MyComponents:MountHole H3
 U 1 1 5C3B6C1C
 P 1350 7700
-F 0 "H?" H 1490 7953 60  0000 L CNN
+F 0 "H3" H 1490 7953 60  0000 L CNN
 F 1 "MountHole" H 1490 7847 60  0000 L CNN
 F 2 "" H 1350 7700 60  0001 C CNN
@@
 $EndComp
 $Comp
-L MyComponents:MountHole H?
+L MyComponents:MountHole H4
 U 1 1 5C3B6C9A
 P 1700 7700
-F 0 "H?" H 1840 7953 60  0000 L CNN
+F 0 "H4" H 1840 7953 60  0000 L CNN
 F 1 "MountHole" H 1840 7847 60  0000 L CNN
 F 2 "" H 1700 7700 60  0001 C CNN
@@
 $EndComp
 $Comp
-L Trigger-rescue:SWD_Pogo-MyComponents U?
+L Trigger-rescue:SWD_Pogo-MyComponents U4
 U 1 1 5C3BB35C
 P 2050 1750
-F 0 "U?" H 1896 2175 50  0000 C CNN
+F 0 "U4" H 1896 2175 50  0000 C CNN
 F 1 "SWD_Pogo" H 1896 2084 50  0000 C CNN
 F 2 "" H 2300 1400 50  0001 C CNN
@@
 Flash
 Text Label 8150 3400 0    50   ~ 0
-Trig
-$Comp
-L Connector:Screw_Terminal_01x06 J?
+Shutter
+$Comp
+L Connector:Screw_Terminal_01x06 J4
 U 1 1 5C3CC01B
 P 7950 3400
-F 0 "J?" H 7870 2875 50  0000 C CNN
+F 0 "J4" H 7870 2875 50  0000 C CNN
 F 1 "Screw_Terminal_01x06" H 7870 2966 50  0000 C CNN
 F 2 "" H 7950 3400 50  0001 C CNN
@@
 $EndComp
 $Comp
-L Connector:Conn_01x04_Female J?
+L Connector:Conn_01x04_Female J3
 U 1 1 5C3D094F
 P 7600 4550
-F 0 "J?" H 7628 4526 50  0000 L CNN
+F 0 "J3" H 7628 4526 50  0000 L CNN
 F 1 "Conn_01x04_IO" H 7628 4435 50  0000 L CNN
 F 2 "" H 7600 4550 50  0001 C CNN
@@
 GND
 $Comp
-L Switch:SW_Push SW?
+L Switch:SW_Push SW2
 U 1 1 5C3E617D
 P 7500 5650
-F 0 "SW?" H 7500 5935 50  0000 C CNN
+F 0 "SW2" H 7500 5935 50  0000 C CNN
 F 1 "SW_Push" H 7500 5844 50  0000 C CNN
 F 2 "" H 7500 5850 50  0001 C CNN
@@
 Text Label 7300 5650 2    50   ~ 0
 ManTrig
-Text Notes 7100 5750 2    50   ~ 0
-To some GPIO
 Text Notes 9050 4550 2    50   ~ 0
 Several GPIOs and Gnd \nAlong edge of board.\nMaybe even more
 $Comp
-L Device:Q_NMOS_GSD Q?
+L Device:Q_NMOS_GSD Q1
 U 1 1 5C3E670E
 P 6950 3350
-F 0 "Q?" H 7155 3396 50  0000 L CNN
+F 0 "Q1" H 7155 3396 50  0000 L CNN
 F 1 "Q_NMOS_GSD" H 7155 3305 50  0000 L CNN
 F 2 "" H 7150 3450 50  0001 C CNN
@@
 $EndComp
 $Comp
-L Device:R R?
+L Device:R R6
 U 1 1 5C3EA1F1
 P 6450 3350
-F 0 "R?" V 6243 3350 50  0000 C CNN
+F 0 "R6" V 6243 3350 50  0000 C CNN
 F 1 "R" V 6334 3350 50  0000 C CNN
 F 2 "" V 6380 3350 50  0001 C CNN
@@
 $EndComp
 $Comp
-L Device:R R?
+L Device:R R5
 U 1 1 5C3EA299
 P 6200 3650
-F 0 "R?" H 6270 3696 50  0000 L CNN
+F 0 "R5" H 6270 3696 50  0000 L CNN
 F 1 "R" H 6270 3605 50  0000 L CNN
 F 2 "" V 6130 3650 50  0001 C CNN
@@
 $EndComp
 $Comp
-L Device:LED_ALT D?
+L Device:LED_ALT D3
 U 1 1 5C3EA341
 P 6200 4000
-F 0 "D?" V 6238 3882 50  0000 R CNN
+F 0 "D3" V 6238 3882 50  0000 R CNN
 F 1 "LED_ALT" V 6147 3882 50  0000 R CNN
 F 2 "" H 6200 4000 50  0001 C CNN
@@
 Wire Wire Line
 	6200 3500 6200 3350
-Connection ~ 6200 3350
 Wire Wire Line
 	6200 3350 6300 3350
@@
 Text Label 6200 4150 2    50   ~ 0
 GND
-Wire Wire Line
-	5400 3350 6200 3350
 Wire Wire Line
 	7050 3550 7050 3700
@@
 Text Notes 7200 3050 2    50   ~ 0
 Pins unlikely to be correct\nfor whatever device actually chosen
+$Comp
+L Connector:Conn_01x01_Male J2
+U 1 1 5C3F95FE
+P 3300 5300
+F 0 "J2" V 3360 5340 50  0000 L CNN
+F 1 "TP1" V 3451 5340 50  0000 L CNN
+F 2 "" H 3300 5300 50  0001 C CNN
+F 3 "~" H 3300 5300 50  0001 C CNN
+	1    3300 5300
+	0    1    1    0
+$EndComp
+Wire Wire Line
+	3000 5550 3300 5550
+Wire Wire Line
+	3300 5550 3300 5500
+Text Label 2900 4050 0    50   ~ 0
+Flash
+Wire Wire Line
+	2900 4050 3200 4050
+Wire Wire Line
+	3200 4150 2900 4150
+Text Label 2900 4150 0    50   ~ 0
+Shutter
+Text Label 2950 3250 0    50   ~ 0
+Trig
+Wire Wire Line
+	2950 3250 3200 3250
+Text Label 4900 5500 0    50   ~ 0
+Trig
+Wire Wire Line
+	3200 3450 3000 3450
+Text Label 3000 3450 2    50   ~ 0
+ManTrig
+Text Label 7400 4550 2    50   ~ 0
+D1
+Text Label 7400 4650 2    50   ~ 0
+D2
+Text Label 7400 4750 2    50   ~ 0
+D3
+Wire Wire Line
+	6000 3550 6000 3350
+Wire Wire Line
+	6000 3350 6200 3350
+Wire Wire Line
+	5400 3550 6000 3550
+Connection ~ 6200 3350
+Text Label 5400 3250 0    50   ~ 0
+D1
+Text Label 5400 3350 0    50   ~ 0
+D2
+Text Label 5400 3450 0    50   ~ 0
+D3
+NoConn ~ 8650 850
+NoConn ~ 1450 3800
+NoConn ~ 3200 3350
+NoConn ~ 3200 3550
+NoConn ~ 3200 3650
+NoConn ~ 3200 3750
+NoConn ~ 3200 3850
+NoConn ~ 3200 3950
+NoConn ~ 3200 4250
+NoConn ~ 3200 4350
+NoConn ~ 3200 4450
+NoConn ~ 3200 4550
+NoConn ~ 5400 4150
+NoConn ~ 5400 4050
+NoConn ~ 5400 3750
+NoConn ~ 5400 3650
 $EndSCHEMATC

Commit message: start parts list
Parts:
- removed R3: 10K, symbol Device:R
- removed SW1: SW_SPST, symbol Switch:SW_SPST
- added C7: 100n, Capacitors_SMD:C_0805_HandSoldering, symbol Device:C_Small
- C1, C2, C3, C4, C6: footprint (none) -> Capacitors_SMD:C_0805_HandSoldering
- C5: value 1u -> 10u; footprint (none) -> Capacitors_SMD:C_0805_HandSoldering
- D1: footprint (none) -> My_Pin_Headers:Pin_Header_Straight_1x02
Connections:
- net GND: now also C7.1
- net RstN: now also C7.2
Changed lines of the file:
@@
 F 0 "U1" H 3041 6253 60  0000 L CNN
 F 1 "MCP6002" H 3041 6147 60  0000 L CNN
-F 2 "" H 2500 6200 60  0000 C CNN
+F 2 "" H 2500 6200 60  0001 C CNN
 F 3 "" H 2500 6200 60  0000 C CNN
 	1    2500 6200
@@
 F 0 "U1" H 4941 6253 60  0000 L CNN
 F 1 "MCP6002" H 4941 6147 60  0000 L CNN
-F 2 "" H 4400 6200 60  0000 C CNN
+F 2 "" H 4400 6200 60  0001 C CNN
 F 3 "" H 4400 6200 60  0000 C CNN
 	2    4400 6200
@@
 F 0 "C1" H 9942 2696 50  0000 R CNN
 F 1 "1u" H 9942 2605 50  0000 L CNN
-F 2 "" H 9850 2650 50  0001 C CNN
+F 2 "Capacitors_SMD:C_0805_HandSoldering" H 9850 2650 50  0001 C CNN
 F 3 "~" H 9850 2650 50  0001 C CNN
 	1    9850 2650
@@
 F 0 "C2" H 10342 2696 50  0000 L CNN
 F 1 "1u" H 10342 2605 50  0000 L CNN
-F 2 "" H 10250 2650 50  0001 C CNN
+F 2 "Capacitors_SMD:C_0805_HandSoldering" H 10250 2650 50  0001 C CNN
 F 3 "~" H 10250 2650 50  0001 C CNN
 	1    10250 2650
@@
 F 0 "C3" H 4265 2396 50  0000 L CNN
 F 1 "1u" H 4265 2305 50  0000 L CNN
-F 2 "" H 4188 2200 50  0001 C CNN
+F 2 "Capacitors_SMD:C_0805_HandSoldering" H 4188 2200 50  0001 C CNN
 F 3 "~" H 4150 2350 50  0001 C CNN
 	1    4150 2350
@@
 F 0 "U3" H 8875 379 60  0000 C CNN
 F 1 "TPS769XX" H 8875 273 60  0000 C CNN
-F 2 "" H 8950 1050 60  0000 C CNN
+F 2 "" H 8950 1050 60  0001 C CNN
 F 3 "" H 8950 1050 60  0000 C CNN
 	1    8950 1050
@@
 P 9900 1000
 F 0 "C5" H 9992 1046 50  0000 L CNN
-F 1 "1u" H 9992 955 50  0000 L CNN
-F 2 "" H 9900 1000 50  0001 C CNN
+F 1 "10u" H 9992 955 50  0000 L CNN
+F 2 "Capacitors_SMD:C_0805_HandSoldering" H 9900 1000 50  0001 C CNN
 F 3 "~" H 9900 1000 50  0001 C CNN
 	1    9900 1000
@@
 F 0 "C4" V 8829 1450 50  0000 C CNN
 F 1 "4u7" V 8738 1450 50  0000 C CNN
-F 2 "" H 8600 1450 50  0001 C CNN
+F 2 "Capacitors_SMD:C_0805_HandSoldering" H 8600 1450 50  0001 C CNN
 F 3 "~" H 8600 1450 50  0001 C CNN
 	1    8600 1450
@@
 Wire Wire Line
 	3750 2550 4150 2550
-$Comp
-L Switch:SW_SPST SW1
-U 1 1 5C3AFA00
-P 4500 2400
-F 0 "SW1" V 4454 2498 50  0000 L CNN
-F 1 "SW_SPST" V 4545 2498 50  0000 L CNN
-F 2 "" H 4500 2400 50  0001 C CNN
-F 3 "~" H 4500 2400 50  0001 C CNN
-	1    4500 2400
-	0    1    1    0
-$EndComp
-Wire Wire Line
-	4150 2200 4500 2200
-Wire Wire Line
-	4500 2650 4500 2600
-$Comp
-L Device:R R3
-U 1 1 5C3B11DD
-P 5200 2400
-F 0 "R3" H 5130 2354 50  0000 R CNN
-F 1 "10K" H 5130 2445 50  0000 R CNN
-F 2 "" V 5130 2400 50  0001 C CNN
-F 3 "~" H 5200 2400 50  0001 C CNN
-	1    5200 2400
-	-1   0    0    1
-$EndComp
 Wire Wire Line
 	4500 2650 5200 2650
@@
 	5200 2650 5200 2550
 Connection ~ 4500 2650
-Text Label 5200 2250 0    50   ~ 0
-3V3
 Wire Wire Line
 	2000 6100 1850 6100
@@
 F 0 "C6" V 2171 5550 50  0000 C CNN
 F 1 "1n" V 2262 5550 50  0000 C CNN
-F 2 "" H 2400 5550 50  0001 C CNN
+F 2 "Capacitors_SMD:C_0805_HandSoldering" H 2400 5550 50  0001 C CNN
 F 3 "~" H 2400 5550 50  0001 C CNN
 	1    2400 5550
@@
 F 0 "D1" V 1404 6357 50  0000 L CNN
 F 1 "D_Photo" V 1495 6357 50  0000 L CNN
-F 2 "" H 1450 6200 50  0001 C CNN
+F 2 "My_Pin_Headers:Pin_Header_Straight_1x02" H 1450 6200 50  0001 C CNN
 F 3 "~" H 1450 6200 50  0001 C CNN
 	1    1500 6200
@@
 NoConn ~ 5400 3750
 NoConn ~ 5400 3650
+$Comp
+L Device:C_Small C7
+U 1 1 5C416F41
+P 4500 2350
+F 0 "C7" H 4592 2396 50  0000 L CNN
+F 1 "100n" H 4592 2305 50  0000 L CNN
+F 2 "Capacitors_SMD:C_0805_HandSoldering" H 4500 2350 50  0001 C CNN
+F 3 "~" H 4500 2350 50  0001 C CNN
+	1    4500 2350
+	1    0    0    -1
+$EndComp
+Wire Wire Line
+	4150 2200 4500 2200
+Wire Wire Line
+	4500 2200 4500 2250
+Wire Wire Line
+	4500 2450 4500 2650
 $EndSCHEMATC

Commit message: more footprints
Parts:
- C1: footprint Capacitors_SMD:C_0805_HandSoldering -> Capacitor_SMD:C_0805_2012Metric
- D2, D3, D4: footprint (none) -> SMD_Mine:LED_SMD_3015
- H1, H2, H3, H4: footprint (none) -> Mount:Hole3
- J2: footprint (none) -> My_Pin_Headers:Pin_Header_Angled_1x01
- J3: footprint (none) -> My_Pin_Headers:Pin_Header_Straight_1x04
- R1, R2, R4, R5, R6, R7, RV1: footprint (none) -> Resistor_SMD:R_0805_2012Metric
Other:
- note added: "LEDs Farnell 2426229 \nKingbright KPL-3051 series"
Changed lines of the file:
@@
 F 0 "C1" H 9942 2696 50  0000 R CNN
 F 1 "1u" H 9942 2605 50  0000 L CNN
-F 2 "Capacitors_SMD:C_0805_HandSoldering" H 9850 2650 50  0001 C CNN
+F 2 "Capacitor_SMD:C_0805_2012Metric" H 9850 2650 50  0001 C CNN
 F 3 "~" H 9850 2650 50  0001 C CNN
 	1    9850 2650
@@
 F 0 "D4" V 10438 883 50  0000 R CNN
 F 1 "LED" V 10347 883 50  0000 R CNN
-F 2 "" H 10400 1000 50  0001 C CNN
+F 2 "SMD_Mine:LED_SMD_3015" H 10400 1000 50  0001 C CNN
 F 3 "~" H 10400 1000 50  0001 C CNN
 	1    10400 1000
@@
 F 0 "R7" V 9943 850 50  0000 C CNN
 F 1 "10K" V 10034 850 50  0000 C CNN
-F 2 "" V 10080 850 50  0001 C CNN
+F 2 "Resistor_SMD:R_0805_2012Metric" V 10080 850 50  0001 C CNN
 F 3 "~" H 10150 850 50  0001 C CNN
 	1    10150 850
@@
 F 0 "R1" V 2193 5200 50  0000 C CNN
 F 1 "100k" V 2284 5200 50  0000 C CNN
-F 2 "" V 2330 5200 50  0001 C CNN
+F 2 "Resistor_SMD:R_0805_2012Metric" V 2330 5200 50  0001 C CNN
 F 3 "~" H 2400 5200 50  0001 C CNN
 	1    2400 5200
@@
 F 0 "RV1" H 3580 6046 50  0000 R CNN
 F 1 "20k" H 3580 5955 50  0000 R CNN
-F 2 "" H 3650 6000 50  0001 C CNN
+F 2 "Resistor_SMD:R_0805_2012Metric" H 3650 6000 50  0001 C CNN
 F 3 "~" H 3650 6000 50  0001 C CNN
 	1    3650 6000
@@
 F 0 "R4" V 5343 6200 50  0000 C CNN
 F 1 "220R" V 5434 6200 50  0000 C CNN
-F 2 "" V 5480 6200 50  0001 C CNN
+F 2 "Resistor_SMD:R_0805_2012Metric" V 5480 6200 50  0001 C CNN
 F 3 "~" H 5550 6200 50  0001 C CNN
 	1    5550 6200
@@
 F 0 "D2" V 5838 6283 50  0000 R CNN
 F 1 "LED" V 5747 6283 50  0000 R CNN
-F 2 "" H 5800 6400 50  0001 C CNN
+F 2 "SMD_Mine:LED_SMD_3015" H 5800 6400 50  0001 C CNN
 F 3 "~" H 5800 6400 50  0001 C CNN
 	1    5800 6400
@@
 F 0 "R2" V 4143 5550 50  0000 C CNN
 F 1 "100k" V 4234 5550 50  0000 C CNN
-F 2 "" V 4280 5550 50  0001 C CNN
+F 2 "Resistor_SMD:R_0805_2012Metric" V 4280 5550 50  0001 C CNN
 F 3 "~" H 4350 5550 50  0001 C CNN
 	1    4350 5550
@@
 F 0 "H1" H 790 7953 60  0000 L CNN
 F 1 "MountHole" H 790 7847 60  0000 L CNN
-F 2 "" H 650 7700 60  0001 C CNN
+F 2 "Mount:Hole3" H 650 7700 60  0001 C CNN
 F 3 "" H 650 7700 60  0001 C CNN
 	1    650  7700
@@
 F 0 "H2" H 1140 7953 60  0000 L CNN
 F 1 "MountHole" H 1140 7847 60  0000 L CNN
-F 2 "" H 1000 7700 60  0001 C CNN
+F 2 "Mount:Hole3" H 1000 7700 60  0001 C CNN
 F 3 "" H 1000 7700 60  0001 C CNN
 	1    1000 7700
@@
 F 0 "H3" H 1490 7953 60  0000 L CNN
 F 1 "MountHole" H 1490 7847 60  0000 L CNN
-F 2 "" H 1350 7700 60  0001 C CNN
+F 2 "Mount:Hole3" H 1350 7700 60  0001 C CNN
 F 3 "" H 1350 7700 60  0001 C CNN
 	1    1350 7700
@@
 F 0 "H4" H 1840 7953 60  0000 L CNN
 F 1 "MountHole" H 1840 7847 60  0000 L CNN
-F 2 "" H 1700 7700 60  0001 C CNN
+F 2 "Mount:Hole3" H 1700 7700 60  0001 C CNN
 F 3 "" H 1700 7700 60  0001 C CNN
 	1    1700 7700
@@
 F 0 "J3" H 7628 4526 50  0000 L CNN
 F 1 "Conn_01x04_IO" H 7628 4435 50  0000 L CNN
-F 2 "" H 7600 4550 50  0001 C CNN
+F 2 "My_Pin_Headers:Pin_Header_Straight_1x04" H 7600 4550 50  0001 C CNN
 F 3 "~" H 7600 4550 50  0001 C CNN
 	1    7600 4550
@@
 F 0 "R6" V 6243 3350 50  0000 C CNN
 F 1 "R" V 6334 3350 50  0000 C CNN
-F 2 "" V 6380 3350 50  0001 C CNN
+F 2 "Resistor_SMD:R_0805_2012Metric" V 6380 3350 50  0001 C CNN
 F 3 "~" H 6450 3350 50  0001 C CNN
 	1    6450 3350
@@
 F 0 "R5" H 6270 3696 50  0000 L CNN
 F 1 "R" H 6270 3605 50  0000 L CNN
-F 2 "" V 6130 3650 50  0001 C CNN
+F 2 "Resistor_SMD:R_0805_2012Metric" V 6130 3650 50  0001 C CNN
 F 3 "~" H 6200 3650 50  0001 C CNN
 	1    6200 3650
@@
 F 0 "D3" V 6238 3882 50  0000 R CNN
 F 1 "LED_ALT" V 6147 3882 50  0000 R CNN
-F 2 "" H 6200 4000 50  0001 C CNN
+F 2 "SMD_Mine:LED_SMD_3015" H 6200 4000 50  0001 C CNN
 F 3 "~" H 6200 4000 50  0001 C CNN
 	1    6200 4000
@@
 F 0 "J2" V 3360 5340 50  0000 L CNN
 F 1 "TP1" V 3451 5340 50  0000 L CNN
-F 2 "" H 3300 5300 50  0001 C CNN
+F 2 "My_Pin_Headers:Pin_Header_Angled_1x01" H 3300 5300 50  0001 C CNN
 F 3 "~" H 3300 5300 50  0001 C CNN
 	1    3300 5300
@@
 Wire Wire Line
 	4500 2450 4500 2650
+Text Notes 8350 6100 0    50   ~ 0
+LEDs Farnell 2426229 \nKingbright KPL-3051 series
 $EndSCHEMATC

Commit message: Finished parts list. Add 5pin header for debug
Parts:
- removed U4: SWD_Pogo, symbol Trigger-rescue:SWD_Pogo-MyComponents
- added J5: Conn_01x05_Male, My_Pin_Headers:Pin_Header_Straight_1x05, symbol Connector:Conn_01x05_Male
- H1, H2, H3, H4: footprint Mount:Hole3 -> My_Pin_Headers:3mm_mount
- J1: footprint (none) -> SMD_Mine:USB_B_Micro_47346-0001
- J4: footprint (none) -> My_Pin_Headers:Screw_6way_3_5mm
- Q1: footprint (none) -> SMD_Mine:SOT-23
- SW2: footprint (none) -> My_Pin_Headers:Tact_SW
- U1: footprint (none) -> SMD_Packages:SOIC-8-N
- U2: footprint (none) -> Housings_QFP:TQFP-32_7x7mm_Pitch0.8mm
- U3: footprint (none) -> SMD_Mine:SOT23_(DBV)
Connections:
- net 3V3: now also J5.2 (Pin_2)
- net GND: now also J5.1 (Pin_1)
- net RstN: now also J5.5 (Pin_5)
- net SWCLK: now also J5.3 (Pin_3)
- net SWDIO: now also J5.4 (Pin_4)
Other:
- note added: "Farnel 1857300 IRLML6346"
- note added: "Farnel 2402398"
- note added: "Farnel 3704610"
Changed lines of the file:
@@
 F 0 "U1" H 3041 6253 60  0000 L CNN
 F 1 "MCP6002" H 3041 6147 60  0000 L CNN
-F 2 "" H 2500 6200 60  0001 C CNN
+F 2 "SMD_Packages:SOIC-8-N" H 2500 6200 60  0001 C CNN
 F 3 "" H 2500 6200 60  0000 C CNN
 	1    2500 6200
@@
 F 0 "U1" H 4941 6253 60  0000 L CNN
 F 1 "MCP6002" H 4941 6147 60  0000 L CNN
-F 2 "" H 4400 6200 60  0001 C CNN
+F 2 "SMD_Packages:SOIC-8-N" H 4400 6200 60  0001 C CNN
 F 3 "" H 4400 6200 60  0000 C CNN
 	2    4400 6200
@@
 F 0 "U3" H 8875 379 60  0000 C CNN
 F 1 "TPS769XX" H 8875 273 60  0000 C CNN
-F 2 "" H 8950 1050 60  0001 C CNN
+F 2 "SMD_Mine:SOT23_(DBV)" H 8950 1050 60  0001 C CNN
 F 3 "" H 8950 1050 60  0000 C CNN
 	1    8950 1050
@@
 F 0 "U2" H 4300 2314 50  0000 C CNN
 F 1 "SAMD21E" H 4300 2223 50  0000 C CNN
-F 2 "" H 4150 4700 50  0001 C CNN
+F 2 "Housings_QFP:TQFP-32_7x7mm_Pitch0.8mm" H 4150 4700 50  0001 C CNN
 F 3 "" H 4150 4700 50  0001 C CNN
 	1    4300 3700
@@
 F 0 "J1" H 1205 4067 50  0000 C CNN
 F 1 "USB_B_Micro" H 1205 3976 50  0000 C CNN
-F 2 "" H 1300 3550 50  0001 C CNN
+F 2 "SMD_Mine:USB_B_Micro_47346-0001" H 1300 3550 50  0001 C CNN
 F 3 "~" H 1300 3550 50  0001 C CNN
 	1    1150 3600
@@
 F 0 "H1" H 790 7953 60  0000 L CNN
 F 1 "MountHole" H 790 7847 60  0000 L CNN
-F 2 "Mount:Hole3" H 650 7700 60  0001 C CNN
+F 2 "My_Pin_Headers:3mm_mount" H 650 7700 60  0001 C CNN
 F 3 "" H 650 7700 60  0001 C CNN
 	1    650  7700
@@
 F 0 "H2" H 1140 7953 60  0000 L CNN
 F 1 "MountHole" H 1140 7847 60  0000 L CNN
-F 2 "Mount:Hole3" H 1000 7700 60  0001 C CNN
+F 2 "My_Pin_Headers:3mm_mount" H 1000 7700 60  0001 C CNN
 F 3 "" H 1000 7700 60  0001 C CNN
 	1    1000 7700
@@
 F 0 "H3" H 1490 7953 60  0000 L CNN
 F 1 "MountHole" H 1490 7847 60  0000 L CNN
-F 2 "Mount:Hole3" H 1350 7700 60  0001 C CNN
+F 2 "My_Pin_Headers:3mm_mount" H 1350 7700 60  0001 C CNN
 F 3 "" H 1350 7700 60  0001 C CNN
 	1    1350 7700
@@
 F 0 "H4" H 1840 7953 60  0000 L CNN
 F 1 "MountHole" H 1840 7847 60  0000 L CNN
-F 2 "Mount:Hole3" H 1700 7700 60  0001 C CNN
+F 2 "My_Pin_Headers:3mm_mount" H 1700 7700 60  0001 C CNN
 F 3 "" H 1700 7700 60  0001 C CNN
 	1    1700 7700
 	1    0    0    -1
 $EndComp
-$Comp
-L Trigger-rescue:SWD_Pogo-MyComponents U4
-U 1 1 5C3BB35C
-P 2050 1750
-F 0 "U4" H 1896 2175 50  0000 C CNN
-F 1 "SWD_Pogo" H 1896 2084 50  0000 C CNN
-F 2 "" H 2300 1400 50  0001 C CNN
-F 3 "" H 2300 1400 50  0001 C CNN
-	1    2050 1750
-	1    0    0    -1
-$EndComp
-Wire Wire Line
-	2050 1550 2200 1550
-Text Label 2200 1550 0    50   ~ 0
-GND
-Wire Wire Line
-	2050 1750 2200 1750
-Wire Wire Line
-	2050 1650 2200 1650
-Wire Wire Line
-	2050 1850 2200 1850
-Wire Wire Line
-	2050 1950 2200 1950
-Text Label 2200 1950 0    50   ~ 0
+Text Label 2900 1500 0    50   ~ 0
+GND
+Text Label 2900 1900 0    50   ~ 0
 RstN
-Text Label 2200 1850 0    50   ~ 0
+Text Label 2900 1700 0    50   ~ 0
 SWCLK
-Text Label 2200 1750 0    50   ~ 0
-3V3
-Text Label 2200 1650 0    50   ~ 0
+Text Label 2900 1600 0    50   ~ 0
+3V3
+Text Label 2900 1800 0    50   ~ 0
 SWDIO
 Text Label 5400 4350 0    50   ~ 0
@@
 F 0 "J4" H 7870 2875 50  0000 C CNN
 F 1 "Screw_Terminal_01x06" H 7870 2966 50  0000 C CNN
-F 2 "" H 7950 3400 50  0001 C CNN
+F 2 "My_Pin_Headers:Screw_6way_3_5mm" H 7950 3400 50  0001 C CNN
 F 3 "~" H 7950 3400 50  0001 C CNN
 	1    7950 3400
@@
 F 0 "SW2" H 7500 5935 50  0000 C CNN
 F 1 "SW_Push" H 7500 5844 50  0000 C CNN
-F 2 "" H 7500 5850 50  0001 C CNN
+F 2 "My_Pin_Headers:Tact_SW" H 7500 5850 50  0001 C CNN
 F 3 "" H 7500 5850 50  0001 C CNN
 	1    7500 5650
@@
 F 0 "Q1" H 7155 3396 50  0000 L CNN
 F 1 "Q_NMOS_GSD" H 7155 3305 50  0000 L CNN
-F 2 "" H 7150 3450 50  0001 C CNN
+F 2 "SMD_Mine:SOT-23" H 7150 3450 50  0001 C CNN
 F 3 "~" H 6950 3350 50  0001 C CNN
 	1    6950 3350
@@
 Text Notes 8350 6100 0    50   ~ 0
 LEDs Farnell 2426229 \nKingbright KPL-3051 series
+Text Notes 6450 2800 0    50   ~ 0
+Farnel 3704610
+Text Notes 6850 3850 0    50   ~ 0
+Farnel 1857300 IRLML6346
+Text Notes 7750 5400 0    50   ~ 0
+Farnel 2402398
+$Comp
+L Connector:Conn_01x05_Male J5
+U 1 1 5C44F716
+P 2700 1700
+F 0 "J5" H 2806 2078 50  0000 C CNN
+F 1 "Conn_01x05_Male" H 2806 1987 50  0000 C CNN
+F 2 "My_Pin_Headers:Pin_Header_Straight_1x05" H 2700 1700 50  0001 C CNN
+F 3 "~" H 2700 1700 50  0001 C CNN
+	1    2700 1700
+	1    0    0    -1
+$EndComp
 $EndSCHEMATC
